File: baseboard.kicad_pcb (KiCad board)
At the start: 2 copper layers, 75.2 x 55.4 mm, 23 parts, among them J1 Conn_01x07, J2 Conn_01x04, P1 CONN_01X09, P2 CONN_01X09, P3 CONN_01X14, P4 CONN_01X14, P5 CONN_01X14, P6 CONN_01X14, P7 CONN_01X02, P8 CONN_01X04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

Commit message: Some changes after HD reorg:
- Fixed the -pro file
- jpg file size change
Other:
- board text added: "+"
- board text added: "-"
Changed lines of the file:
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@@
-(kicad_pcb (version 4) (host pcbnew 4.0.7-e2-6376~58~ubuntu15.04.1)
+(kicad_pcb (version 4) (host pcbnew 4.0.5+dfsg1-4)
   (general
     (links 120)
@@
     (area 70.375 88.549 148.543334 148.975001)
     (thickness 1.6)
-    (drawings 48)
+    (drawings 50)
     (tracks 191)
     (zones 0)
@@
     )
   )
+  (gr_text - (at 104.775 96.52) (layer F.Fab)
+    (effects (font (size 1.5 1.5) (thickness 0.3)))
+  )
+  (gr_text + (at 113.03 96.52) (layer F.Fab)
+    (effects (font (size 1.5 1.5) (thickness 0.3)))
+  )
   (gr_line (start 140.97 99.822) (end 141.224 99.822) (angle 90) (layer F.SilkS) (width 0.2))
   (gr_line (start 140.97 98.298) (end 140.97 99.822) (angle 90) (layer F.SilkS) (width 0.2))
   (gr_line (start 118.11 98.298) (end 140.97 98.298) (angle 90) (layer F.SilkS) (width 0.2))
   (gr_line (start 140.97 98.298) (end 140.97 100.33) (angle 90) (layer F.Fab) (width 0.2))
-  (gr_line (start 118.11 98.298) (end 140.97 98.298) (angle 90) (layer F.Fab) (width 0.2))
+  (gr_line (start 118.11 98.298) (end 140.97 98.298) (angle 90) (layer F.Fab) (width 0.3))
   (gr_line (start 133.858 141.097) (end 140.97 133.985) (angle 90) (layer F.SilkS) (width 0.2))
   (gr_line (start 124.968 141.097) (end 133.858 141.097) (angle 90) (layer F.SilkS) (width 0.2))
   (gr_line (start 118.11 134.239) (end 124.968 141.097) (angle 90) (layer F.SilkS) (width 0.2))
   (gr_line (start 124.968 141.097) (end 124.46 140.589) (angle 90) (layer F.Fab) (width 0.2))
-  (gr_line (start 133.858 141.097) (end 124.968 141.097) (angle 90) (layer F.Fab) (width 0.2))
-  (gr_line (start 140.97 133.985) (end 133.858 141.097) (angle 90) (layer F.Fab) (width 0.2))
-  (gr_line (start 118.11 134.239) (end 124.46 140.589) (angle 90) (layer F.Fab) (width 0.2))
+  (gr_line (start 133.858 141.097) (end 124.968 141.097) (angle 90) (layer F.Fab) (width 0.3))
+  (gr_line (start 140.97 133.985) (end 133.858 141.097) (angle 90) (layer F.Fab) (width 0.3))
+  (gr_line (start 118.11 134.239) (end 124.46 140.589) (angle 90) (layer F.Fab) (width 0.3))
   (gr_line (start 129.794 96.266) (end 124.714 96.266) (angle 90) (layer F.SilkS) (width 0.2))
   (gr_line (start 129.794 91.313) (end 129.794 96.139) (angle 90) (layer F.SilkS) (width 0.2))
@@
   (gr_line (start 128.016 142.367) (end 134.62 142.367) (angle 90) (layer F.Fab) (width 0.2))
   (gr_line (start 128.016 144.145) (end 128.016 142.367) (angle 90) (layer F.Fab) (width 0.2))
-  (gr_line (start 135.89 144.78) (end 135.89 133.35) (angle 90) (layer F.Fab) (width 0.2))
-  (gr_line (start 118.11 144.78) (end 135.89 144.78) (angle 90) (layer F.Fab) (width 0.2))
-  (gr_line (start 118.11 133.35) (end 118.11 144.78) (angle 90) (layer F.Fab) (width 0.2))
-  (gr_line (start 135.89 90.678) (end 135.89 100.33) (angle 90) (layer F.Fab) (width 0.2))
-  (gr_line (start 118.11 90.678) (end 135.89 90.678) (angle 90) (layer F.Fab) (width 0.2))
-  (gr_line (start 118.11 100.33) (end 118.11 90.678) (angle 90) (layer F.Fab) (width 0.2))
+  (gr_line (start 135.89 144.78) (end 135.89 133.35) (angle 90) (layer F.Fab) (width 0.3))
+  (gr_line (start 118.11 144.78) (end 135.89 144.78) (angle 90) (layer F.Fab) (width 0.3))
+  (gr_line (start 118.11 133.35) (end 118.11 144.78) (angle 90) (layer F.Fab) (width 0.3))
+  (gr_line (start 135.89 90.678) (end 135.89 100.33) (angle 90) (layer F.Fab) (width 0.3))
+  (gr_line (start 118.11 90.678) (end 135.89 90.678) (angle 90) (layer F.Fab) (width 0.3))
+  (gr_line (start 118.11 100.33) (end 118.11 90.678) (angle 90) (layer F.Fab) (width 0.3))
   (gr_circle (center 127.254 93.726) (end 128.778 92.456) (layer F.Fab) (width 0.2))
   (gr_line (start 135.89 133.35) (end 136.144 133.35) (angle 90) (layer F.Fab) (width 0.2))
